Commit message: modified:   src/moveit_config/config/simple_moveit_controllers.yaml 	modified:   src/moveit_config/launch/demo.launch 	modified:   src/moveit_config/launch/gazebo.launch 	modified:   src/moveit_config/launch/moveit.rviz 	modified:   src/moveit_config/launch/trajectory_execution.launch.xml

File: src/abb_robot/urdf/abb_robot_description.urdf (robot description, URDF)
Before this commit: robot homos, 8 links, 7 joints
Links:
- added link world
- link base: mass None -> 0.1
- link end_effector: mass None -> 0.1
- link link_1: mass None -> 0.1
- link link_2: mass None -> 0.1
- link link_3: mass None -> 0.1
- link link_4: mass None -> 0.1
- link link_5: mass None -> 0.1
- link link_6: mass None -> 0.1
Joints:
- added joint world_joint: type fixed, parent world, child base, origin xyz=0 0 0.1 rpy=0 0 0, axis 0 0 0
